Commit message: Changed urdf to have textures

File: robofin/urdf/franka_panda/panda_deprecated.urdf (robot description, URDF)
Before this commit: robot panda, 14 links, 13 joints
Links:
- link panda_hand: geometry collision mesh filename=meshes/collision/hand.stl; visual mesh filename=meshes/visual/hand.dae
- link panda_leftfinger: geometry collision mesh filename=meshes/collision/finger.stl; visual mesh filename=meshes/visual/finger.dae
- link panda_link0: geometry collision mesh filename=meshes/collision/link0.stl; visual mesh filename=meshes/visual/link0.dae
- link panda_link1: geometry collision mesh filename=meshes/collision/link1.stl; visual mesh filename=meshes/visual/link1.dae
- link panda_link2: geometry collision mesh filename=meshes/collision/link2.stl; visual mesh filename=meshes/visual/link2.dae
- link panda_link3: geometry collision mesh filename=meshes/collision/link3.stl; visual mesh filename=meshes/visual/link3.dae
- link panda_link4: geometry collision mesh filename=meshes/collision/link4.stl; visual mesh filename=meshes/visual/link4.dae
- link panda_link5: geometry collision mesh filename=meshes/collision/link5.stl; visual mesh filename=meshes/visual/link5.dae
- link panda_link6: geometry collision mesh filename=meshes/collision/link6.stl; visual mesh filename=meshes/visual/link6.dae
- link panda_link7: geometry collision mesh filename=meshes/collision/link7.stl; visual mesh filename=meshes/visual/link7.dae
- link panda_rightfinger: geometry collision mesh filename=meshes/collision/finger.stl; visual mesh filename=meshes/visual/finger.dae
Joints:
- joint panda_joint1: limit lower=-2.9671 upper=2.9671 effort=87 velocity=2.1750 -> lower=-2.8973 upper=2.8973 effort=87 velocity=2.1750
- joint panda_joint2: limit lower=-1.8326 upper=1.8326 effort=87 velocity=2.1750 -> lower=-1.7628 upper=1.7628 effort=87 velocity=2.1750
- joint panda_joint3: limit lower=-2.9671 upper=2.9671 effort=87 velocity=2.1750 -> lower=-2.8973 upper=2.8973 effort=87 velocity=2.1750
- joint panda_joint4: limit lower=-3.1416 upper=0.0 effort=87 velocity=2.1750 -> lower=-3.0718 upper=-0.0698 effort=87 velocity=2.1750
- joint panda_joint5: limit lower=-2.9671 upper=2.9671 effort=12 velocity=2.6100 -> lower=-2.8973 upper=2.8973 effort=12 velocity=2.6100
- joint panda_joint6: limit lower=-0.0873 upper=3.8223 effort=12 velocity=2.6100 -> lower=-0.0175 upper=3.7525 effort=12 velocity=2.6100
- joint panda_joint7: limit lower=-2.9671 upper=2.9671 effort=12 velocity=2.6100 -> lower=-2.8973 upper=2.8973 effort=12 velocity=2.6100
