Commit message: Updated meshes in panda hand

File: robofin/urdf/panda_hand/panda.urdf (robot description, URDF)
Before this commit: robot panda_hand, 10 links, 9 joints
Links:
- link panda_hand: geometry collision mesh filename=meshes/collision/hand.stl; visual mesh filename=meshes/visual/hand.obj
- link panda_leftfinger: geometry collision mesh filename=meshes/collision/finger.stl; visual mesh filename=meshes/visual/finger.obj
- link panda_rightfinger: geometry collision mesh filename=meshes/collision/finger.stl; visual mesh filename=meshes/visual/finger.obj
